File: deltaAY.kicad_sch (KiCad schematic)
At the start: 0 parts

Commit message: 31 may 2023
Parts:
- added C1, C2: 10uF 5V, Capacitor_THT:CP_Radial_D8.0mm_P3.80mm, symbol Device:C_Polarized
- added D1: ~, Package_DIP:DIP-40_W15.24mm_LongPads, symbol deltaAY_symbols:AY-3-8910
- added J1: SNP, deltaAY:SNP96, symbol deltaAY_symbols:SNP
- added J2: Jack_3.5mm_5pin, deltaAY:jack_5_pin_3f07_FINAL, symbol deltaAY_symbols:AudioJack_5_pin
- added R1, R2: 330, Resistor_THT:R_Axial_DIN0207_L6.3mm_D2.5mm_P7.62mm_Horizontal, symbol Device:R
- added R3, R4, R5, R6, R7, R8: 2K, Resistor_THT:R_Axial_DIN0207_L6.3mm_D2.5mm_P7.62mm_Horizontal, symbol Device:R
- added U1: М555ЛН1 (SN74LS04), Package_DIP:DIP-14_W7.62mm_LongPads, symbol 74xx:74LS04
- added U2: К555ТМ2 (SN74LS74), Package_DIP:DIP-14_W7.62mm_LongPads, symbol 74xx:74LS74
- added U3: К555ЛЛ1 (SN74LS32), Package_DIP:DIP-14_W7.62mm_LongPads, symbol 74xx:74LS32
- added U4: К555ЛЕ1 (SN74LS02), Package_DIP:DIP-14_W7.62mm_LongPads, symbol 74xx:74LS02
- added Y1: 3.579545Mhz, Crystal:Crystal_HC49-U_Horizontal, symbol Device:Crystal
Connections:
- new net: U3.3, U4.3, U4.5
- new net: U3.6, U4.6
- new net: R1.1, U1.1, Y1.1
- new net: R1.2, R2.1, U1.2, U1.3
- new net: C1.1, R3.2, R6.2, R7.2
- new net: U3.4, U4.10
- new net: U3.5, U4.13
- new net: U2.2 (D), U2.6 (~{Q})
- new net: R2.2, U1.4, U2.3 (C), Y1.2
- new net: C2.1, R4.2, R5.2, R8.1
- new net: C1.2, J2.5
- new net: C2.2, J2.2
- new net +5V: D1.25 (A8), D1.28 (BC2), D1.40 (VCC), J1.35 ("+5"), J1.47 ("+5"), J1.48 ("+5"), U1.14 (VCC), U2.1 (~{R}), U2.14 (VCC), U2.4 (~{S}), U3.14 (VCC), U4.14 (VCC)
- new net A1: J1.41 (A1), U3.2
- new net A14: J1.33 (A14), U4.8, U4.9
- new net AY22: D1.22 (CLOCK), U2.5 (Q)
- new net AY27: D1.27 (BDIR), U4.1
- new net AY29: D1.29 (BC1), U4.4
- new net AY_A: D1.4 (analog_A), R3.1
- new net AY_B: D1.3 (analog_B), R5.1, R6.1
- new net AY_C: D1.38 (analog_C), R4.1
- new net DA0: D1.37 (DA0), J1.5 (D0)
- new net DA1: D1.36 (DA1), J1.6 (D1)
- new net DA2: D1.35 (DA2), J1.7 (D2)
- new net DA3: D1.34 (DA3), J1.10 (D3)
- new net DA4: D1.33 (DA4), J1.11 (D4)
- new net DA5: D1.32 (DA5), J1.9 (D5)
- new net DA6: D1.31 (DA6), J1.8 (D6)
- new net DA7: D1.30 (DA7), J1.3 (D7)
- new net GND: D1.1 (GND), D1.24 (A9), J1.37 (Общий), J1.38 (Общий), J1.45 (Общий), J2.1, R7.1, R8.2, U1.7 (GND), U2.7 (GND), U3.7 (GND), U4.7 (GND)
- new net IORQ: J1.16 (ВУ), U3.1
- new net M1: J1.23 (М1), U4.11, U4.12
- new net RESET: D1.23 (RESET), J1.27 (СБРОС)
- new net WR: J1.18 (ЗП), U4.2
- no-connect marks 0 -> 59

Commit message: Update 19072023
Parts:
- J1: value SNP -> СНП59-96
- U4: renamed from D1; value ~ -> AY-3-8910
- renumbered R2 to R1, R1 to R2, R7 to R3, R6 to R4, R3 to R5, R4 to R6, R5 to R7, U3 to U1, U4 to U2, U2 to U3, U1 to U5

Commit message: Release ver1 19-07-2023
First release
Parts:
- C1, C2: value 10uF 5V -> 10μF 5V
- R3, R4, R7, R8: value 2K -> 2K/2.2K
- R5, R6: value 2K -> 2K/1K
Changed lines of the file:
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@@
       (effects (font (size 1.27 1.27)))
     )
-    (property "Value" "2K" (at 38.1 109.22 90)
+    (property "Value" "2K/1K" (at 38.1 109.22 90)
       (effects (font (size 1.27 1.27)))
     )
@@
       (effects (font (size 1.27 1.27)))
     )
-    (property "Value" "2K" (at 66.04 101.6 90)
+    (property "Value" "2K/2.2K" (at 66.04 101.6 90)
       (effects (font (size 1.27 1.27)))
     )
@@
       (effects (font (size 1.27 1.27)))
     )
-    (property "Value" "2K" (at 54.61 118.11 90)
+    (property "Value" "2K/2.2K" (at 54.61 118.11 90)
       (effects (font (size 1.27 1.27)))
     )
@@
       (effects (font (size 1.27 1.27)))
     )
-    (property "Value" "10uF 5V" (at 79.121 105.41 90)
+    (property "Value" "10μF 5V" (at 79.121 105.41 90)
       (effects (font (size 1.27 1.27)))
     )
@@
       (effects (font (size 1.27 1.27)))
     )
-    (property "Value" "2K" (at 54.61 113.03 90)
+    (property "Value" "2K/2.2K" (at 54.61 113.03 90)
       (effects (font (size 1.27 1.27)))
     )
@@
       (effects (font (size 1.27 1.27)))
     )
-    (property "Value" "10uF 5V" (at 79.121 118.11 90)
+    (property "Value" "10μF 5V" (at 79.121 118.11 90)
       (effects (font (size 1.27 1.27)))
     )
@@
       (effects (font (size 1.27 1.27)))
     )
-    (property "Value" "2K" (at 66.04 129.54 90)
+    (property "Value" "2K/2.2K" (at 66.04 129.54 90)
       (effects (font (size 1.27 1.27)))
     )
@@
       (effects (font (size 1.27 1.27)))
     )
-    (property "Value" "2K" (at 38.1 121.92 90)
-      (effects (font (size 1.27 1.27)))
-    )
+    (property "Value" "2K/1K" (at 38.1 121.92 90)
+      (effects (font (size 1.27 1.27)))
+    )
